File: dcf77_clock.brd (EAGLE design)
At the start: 83.1 x 76.2 mm, 42 parts, among them IC1 DS1307SO8, IC2 7805DT, IC3 ATMEGA48/88/168-AU, J1 DCJ0202, Q1 32.768kHz, Q2 IRLML6244TRPBF, SW1 EC12E_SW, U1 AVR_SPI_PROG2PTH2, U2 LCD-16X2UPPERHOLES

Commit message: Add 3V3 LDO and level shifter for MAS6181B
Parts:
- added C11, C12: 1u, rcl:C0805K
- added IC4: DI62063.3S2, dcf77:SOT23
- added Q3: IRLML6244TRPBF, sosbutton:SOT23
- added R13, R14: 10k, rcl:M0805
- R1: value 4.7k -> 10k
- moved C5 2.77 mm to (40.6, 53.7)
- moved Q2 2.29 mm to (46.1, 58.3)
- moved R6 1.91 mm to (48.9, 59.6)
- moved R7 1.65 mm to (51.1, 59.6)
- moved C2 1.57 mm to (33.7, 59.7)
- moved C9 1.52 mm to (53.1, 59.6)
- moved D1 1.49 mm to (45.8, 55.1)
- moved C7 1.27 mm to (34.2, 51.7)
- moved Q1 1.14 mm to (28.3, 59.2)
- moved R8 1.02 mm to (55.1, 59.6)
- moved C10 0.51 mm to (57.1, 59.6)
Connections:
- new net +3V3: C12.1, C2.1, IC4.2, MOD1.P$5, R14.2
- new net N$6: MOD1.P$2, Q3.1
- net DCF77_OUT: now also Q3.3, R13.1; no longer MOD1.P$2
- net DCF77_SEL: now also R14.1
- net GND: now also C11.2, C12.2, IC4.1, Q3.2
- net VCC: now also C11.1, IC4.3, R13.2; no longer C2.1, MOD1.P$5
Routing:
- net N$6: track 0.00 -> 13.7 mm, vias 0 -> 1
- net +3V3: track 0.00 -> 9.53 mm
- net VCC: track 242.0 -> 234.1 mm
- net DCF77_OUT: track 25.2 -> 19.1 mm, vias 1 -> 2
- net DCF77_SEL: track 24.9 -> 28.1 mm, vias 1 -> 2
- net ISP_MOSI_BUZ_PWM: track 55.6 -> 53.3 mm
- net N$2: track 8.78 -> 7.08 mm
- net N$10: track 25.0 -> 23.9 mm
- net N$11: track 27.2 -> 26.1 mm
- net N$3: track 4.96 -> 4.33 mm
- net ENC_B: track 53.4 -> 52.9 mm
Other:
- board text added: "DCF77 CLOCK AWESOMETRONICS"
- board text removed: "DCF77 Clock AWESOMETRONICS"
