File: dcf77_clock.brd (EAGLE design)
At the start: 83.1 x 76.2 mm, 48 parts, among them IC1 DS1307SO8, IC2 7805DT, IC3 ATMEGA48/88/168-AU, IC4 DI62063.3S2, J1 DCJ0202, Q1 32.768kHz, Q2 IRLML6244TRPBF, Q3 IRLML6244TRPBF, SW1 EC12E_SW, U1 AVR_SPI_PROG2PTH2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

Commit message: Fix CR2032 holder footprint
Routing:
- net N$12: track 20.1 -> 19.2 mm
Changed lines of the file:
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@@
 <wire x1="2.54" y1="63.5" x2="1.27" y2="63.5" width="0.4064" layer="1"/>
 <wire x1="1.27" y1="63.5" x2="0.635" y2="62.865" width="0.4064" layer="1"/>
-<wire x1="0.635" y1="54.008" x2="4.986" y2="49.657" width="0.4064" layer="1"/>
+<wire x1="0.635" y1="51.908" x2="2.886" y2="49.657" width="0.4064" layer="1"/>
 <wire x1="3.175" y1="64.135" x2="2.54" y2="63.5" width="0.4064" layer="1"/>
-<wire x1="0.635" y1="62.865" x2="0.635" y2="54.008" width="0.4064" layer="1"/>
+<wire x1="0.635" y1="62.865" x2="0.635" y2="51.908" width="0.4064" layer="1"/>
 </signal>
 <signal name="RTC_SQW">

Commit message: Change LED resistor to limit brightness
Parts:
- R10: value 100R -> 330R
Changed lines of the file:
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@@
 <attribute name="VALUE" x="46.355" y="60.833" size="1.27" layer="27" rot="R270"/>
 </element>
-<element name="R10" library="rcl" library_urn="urn:adsk.eagle:library:334" package="M0805" package3d_urn="urn:adsk.eagle:package:23556/2" value="100R" x="44.45" y="38.989" smashed="yes" rot="R180">
+<element name="R10" library="rcl" library_urn="urn:adsk.eagle:library:334" package="M0805" package3d_urn="urn:adsk.eagle:package:23556/2" value="330R" x="44.45" y="38.989" smashed="yes" rot="R180">
 <attribute name="NAME" x="42.164" y="39.37" size="1.27" layer="25" rot="R180"/>
 <attribute name="POPULARITY" value="45" x="44.45" y="38.989" size="1.778" layer="27" rot="R180" display="off"/>
